Commit message: 添加自定义消息抓取

File: src/realsense-ros/realsense2_description/urdf/test_d415_camera.urdf.xacro (robot description, xacro)
@@ -5,7 +5,7 @@
   <xacro:arg name="use_mesh" default="true" />
   <xacro:include filename="$(find realsense2_description)/urdf/_d415.urdf.xacro" />
-  <link name="base_link" />
-  <xacro:sensor_d415 parent="base_link" use_nominal_extrinsics="$(arg use_nominal_extrinsics)" add_plug="$(arg add_plug)" use_mesh="$(arg use_mesh)">
+  <!-- <link name="base_link" /> -->
+  <!-- <xacro:sensor_d415 parent="Link6" use_nominal_extrinsics="$(arg use_nominal_extrinsics)" add_plug="$(arg add_plug)" use_mesh="$(arg use_mesh)">
     <origin xyz="0 0 0" rpy="0 0 0"/>
-  </xacro:sensor_d415>
+  </xacro:sensor_d415> -->
 </robot>

File: src/rm_robot/rm_description/urdf/RM65/rm_65.urdf.xacro (robot description, xacro)
@@ -445,4 +445,9 @@
 	<dynamics damping="50" friction="1"/>
   </joint>
+  <!-- <xacro:arg name="use_nominal_extrinsics" default="false"/>
+  <xacro:include filename="$(find realsense2_description)/urdf/_d415.urdf.xacro" />
+  <xacro:sensor_d415 parent="Link6" use_nominal_extrinsics="$(arg use_nominal_extrinsics)" >
+      <origin xyz="0.0 0.06 0.05" rpy="0 0 1.57"/>
+  </xacro:sensor_d415>  -->
   <!-- Transmissions for ROS Control -->
   <xacro:macro name="transmission_block" params="joint_name">

Commit message: 合并基准1

File: src/realsense-ros/realsense2_description/urdf/test_d415_camera.urdf.xacro (robot description, xacro)
@@ -5,7 +5,7 @@
   <xacro:arg name="use_mesh" default="true" />
   <xacro:include filename="$(find realsense2_description)/urdf/_d415.urdf.xacro" />
-  <!-- <link name="base_link" /> -->
-  <!-- <xacro:sensor_d415 parent="Link6" use_nominal_extrinsics="$(arg use_nominal_extrinsics)" add_plug="$(arg add_plug)" use_mesh="$(arg use_mesh)">
+  <link name="base_link" />
+  <xacro:sensor_d415 parent="base_link" use_nominal_extrinsics="$(arg use_nominal_extrinsics)" add_plug="$(arg add_plug)" use_mesh="$(arg use_mesh)">
     <origin xyz="0 0 0" rpy="0 0 0"/>
-  </xacro:sensor_d415> -->
+  </xacro:sensor_d415>
 </robot>
