Commit message: urdf+抓取测试

File: src/rm_robot/rm_description/urdf/sensors/_d415.urdf.xacro (robot description, xacro)
@@ -36,10 +36,10 @@
     </joint>
     <link name="${name}_bottom_screw_frame"/>
-    <joint name="${name}_link_joint" type="fixed">
+    <joint name="${name}_link1_joint" type="fixed">
       <origin xyz="0 ${d415_cam_depth_py} ${d415_cam_depth_pz}" rpy="0 0 0"/>
       <parent link="${name}_bottom_screw_frame"/>
-      <child link="${name}_link" />
+      <child link="${name}_link1" />
     </joint>
-    <link name="${name}_link">
+    <link name="${name}_link1">
       <visual>
         <xacro:if value="${use_mesh}">
@@ -75,5 +75,5 @@
       <joint name="${name}_depth_joint" type="fixed">
         <origin xyz="0 0 0" rpy="0 0 0"/>
-        <parent link="${name}_link"/>
+        <parent link="${name}_link1"/>
         <child link="${name}_depth_frame" />
       </joint>
@@ -88,5 +88,5 @@
       <joint name="${name}_infra1_joint" type="fixed">
         <origin xyz="0 ${d415_cam_depth_to_infra1_offset} 0" rpy="0 0 0" />
-        <parent link="${name}_link" />
+        <parent link="${name}_link1" />
         <child link="${name}_infra1_frame" />
       </joint>
@@ -101,5 +101,5 @@
       <joint name="${name}_infra2_joint" type="fixed">
         <origin xyz="0 ${d415_cam_depth_to_infra2_offset} 0" rpy="0 0 0" />
-        <parent link="${name}_link" />
+        <parent link="${name}_link1" />
         <child link="${name}_infra2_frame" />
       </joint>
@@ -114,5 +114,5 @@
       <joint name="${name}_color_joint" type="fixed">
         <origin xyz="0 ${d415_cam_depth_to_color_offset} 0" rpy="0 0 0" />
-        <parent link="${name}_link" />
+        <parent link="${name}_link1" />
         <child link="${name}_color_frame" />
       </joint>
@@ -126,5 +126,5 @@
     </xacro:if>
     <xacro:if value="${add_plug}">
-      <xacro:usb_plug parent="${name}_link" name="${name}_usb_plug">
+      <xacro:usb_plug parent="${name}_link1" name="${name}_usb_plug">
         <origin xyz="${d415_cam_mount_from_center_offset - 0.01587} ${-d415_cam_depth_py - 0.0358} 0" rpy="0 0 0"/>
       </xacro:usb_plug>
