Commit message: 1

File: src/rm_robot/rm_moveit_config/rm_65_moveit_config/config/gazebo_rm_65.urdf (robot description, URDF)
Before this commit: robot rm_65, 16 links, 15 joints
Links:
- removed link camera_link
- added link camera_link1, mass 0.072; collision box size=0.02005 0.099 0.023; visual mesh filename=package://realsense2_description/meshes/d415.stl
Joints:
- removed joint camera_link_joint
- added joint camera_link1_joint: type fixed, parent camera_bottom_screw_frame, child camera_link1, origin xyz=0 0.02 0.0115 rpy=0 0 0
- joint joint_ee_link: origin xyz=0 0 0.15 rpy=0 0 0 -> xyz=0 0 0.14 rpy=0 0 0
- joint joint_tool0: origin xyz=0 0 0.01 rpy=0 0 0 -> xyz=0 0 0.015 rpy=0 0 0
