Commit message: add car model

File: src/rm_robot/rm_description/urdf/RM65/rm_65_add.urdf.xacro (robot description, xacro)
@@ -493,54 +493,4 @@
       <child link="gripper_link" />
     </joint>
-    <!-- finger1 -->
-    <link name="finger1">
-      <visual>
-        <origin xyz="0 0 0.0325" rpy="0 0 0"/>
-        <material
-          name="">
-          <color
-            rgba="1 1 1 1" />
-        </material>
-        <geometry>
-            <box size="0.046 0.003 0.065"/>
-        </geometry>
-      </visual>
-      <collision>
-        <origin xyz="0 0 0.0325" rpy="0 0 0"/>
-        <geometry>
-            <box size="0.046 0.003 0.065"/>
-        </geometry>
-      </collision>
-    </link>
-    <joint name="joint_finger1" type="fixed">
-      <origin xyz="0 0.0265 0.11" rpy="0 0 0" />
-      <parent link="gripper_link" />
-      <child link="finger1" />
-    </joint>
-    <!-- finger2 -->
-    <link name="finger2">
-      <visual>
-        <origin xyz="0 0 0.0325" rpy="0 0 0"/>
-        <material
-          name="">
-          <color
-            rgba="1 1 1 1" />
-        </material>
-        <geometry>
-            <box size="0.046 0.003 0.065"/>
-        </geometry>
-      </visual>
-      <collision>
-        <origin xyz="0 0 0.0325" rpy="0 0 0"/>
-        <geometry>
-            <box size="0.046 0.003 0.065"/>
-        </geometry>
-      </collision>
-    </link>
-    <joint name="joint_finger2" type="fixed">
-      <origin xyz="0 -0.0265 0.11" rpy="0 0 0" />
-      <parent link="gripper_link" />
-      <child link="finger2" />
-    </joint>
     <!-- Transmissions for ROS Control -->
     <xacro:macro name="transmission_block" params="joint_name">

File: src/rm_robot/rm_description/urdf/RM65/rm_65_plus.urdf.xacro (robot description, xacro)
@@ -448,11 +448,4 @@
 	<dynamics damping="50" friction="1"/>
   </joint>
-  <!-- tool -->
-  <link name="tool0"/>
-  <joint name="joint_tool0" type="fixed">
-    <origin xyz="0 0 0.015" rpy="0 0 0" />
-    <parent link="Link6" />
-    <child link="tool0" />
-  </joint>
   <!-- tool_frame -->
   <link name="ee_link"/>
@@ -463,9 +456,9 @@
   </joint>
   <!-- camera -->
-  <xacro:include filename="$(find rm_description)/urdf/sensors/_d415.urdf.xacro"/>
+  <!-- <xacro:include filename="$(find rm_description)/urdf/sensors/_d415.urdf.xacro"/>
     <xacro:sensor_d415  parent="tool0">
         <origin xyz="-0.05 0 0"
                 rpy="0 -1.57 0" />
-  </xacro:sensor_d415>
+  </xacro:sensor_d415> -->
   <!-- gripper -->
   <link name="gripper_link">
@@ -489,10 +482,10 @@
   </link>
   <joint name="joint_gripper" type="fixed">
-    <origin xyz="0 0 0" rpy="0 0 0" />
-    <parent link="tool0" />
+    <origin xyz="0 0 0.015" rpy="0 0 0" />
+    <parent link="Link6" />
     <child link="gripper_link" />
   </joint>
   <!-- finger1 -->
-  <link name="finger1">
+  <!-- <link name="finger1">
     <visual>
       <origin xyz="0 0 0.0325" rpy="0 0 0"/>
@@ -517,7 +510,7 @@
     <parent link="gripper_link" />
     <child link="finger1" />
-  </joint>
+  </joint> -->
   <!-- finger2 -->
-  <link name="finger2">
+  <!-- <link name="finger2">
     <visual>
       <origin xyz="0 0 0.0325" rpy="0 0 0"/>
@@ -542,5 +535,5 @@
     <parent link="gripper_link" />
     <child link="finger2" />
-  </joint>
+  </joint> -->
   <!-- Transmissions for ROS Control -->
   <xacro:macro name="transmission_block" params="joint_name">

File: src/rm_robot/rm_moveit_config/rm_65_moveit_config/config/gazebo_base.urdf (robot description, URDF)
Before this commit: robot rm_65, 10 links, 9 joints
Links:
- removed link world
- added link back_l, mass 0.1; collision cylinder length=0.015 radius=0.035; visual cylinder length=0.015 radius=0.035
- added link back_r, mass 0.1; collision cylinder length=0.015 radius=0.035; visual cylinder length=0.015 radius=0.035
- added link base_link, mass 0.1; collision cylinder length=0.26 radius=0.23; visual cylinder length=0.26 radius=0.23
- added link front_l, mass 0.1; collision cylinder length=0.015 radius=0.035; visual cylinder length=0.015 radius=0.035
- added link front_r, mass 0.1; collision cylinder length=0.015 radius=0.035; visual cylinder length=0.015 radius=0.035
- added link left_wheel_link, mass 0.1; collision cylinder length=0.06 radius=0.07; visual cylinder length=0.06 radius=0.07
- added link right_wheel_link, mass 0.1; collision cylinder length=0.06 radius=0.07; visual cylinder length=0.06 radius=0.07
- added link tool0
Joints:
- added joint back_l_caster_joint: type fixed, parent base_link, child back_l, origin xyz=0.14 0.07 -0.035 rpy=1.5707963 0 0, axis 0 1 0
- added joint back_r_caster_joint: type fixed, parent base_link, child back_r, origin xyz=-0.14 -0.07 -0.035 rpy=1.5707963 0 0, axis 0 1 0
- added joint front_l_caster_joint: type fixed, parent base_link, child front_l, origin xyz=0.14 -0.07 -0.035 rpy=1.5707963 0 0, axis 0 1 0
- added joint front_r_caster_joint: type fixed, parent base_link, child front_r, origin xyz=-0.14 0.07 -0.035 rpy=1.5707963 0 0, axis 0 1 0
- added joint joint_tool0: type fixed, parent Link6, child tool0, origin xyz=0 0 0.015 rpy=0 0 0
- added joint left_wheel_joint: type fixed, parent base_link, child left_wheel_link, origin xyz=0 0.19 0 rpy=1.5707963 0 0, axis 0 1 0
- added joint right_wheel_joint: type fixed, parent base_link, child right_wheel_link, origin xyz=0 -0.19 0 rpy=1.5707963 0 0, axis 0 1 0
- joint dummy_joint: origin (none) -> xyz=0.135 0.0 0.26 rpy=0.0 0.0 0.0; parent world -> base_link
- joint joint_gripper: origin xyz=0 0 0.015 rpy=0 0 0 -> xyz=0 0 0 rpy=0 0 0; parent Link6 -> tool0

Commit message: 上传opencabinate

File: src/rm_robot/rm_description/urdf/RM65/rm_65_add.urdf.xacro (robot description, xacro)
@@ -449,10 +449,10 @@
     </joint>
     <!-- tool -->
-    <link name="tool0"/>
+    <!-- <link name="tool0"/>
     <joint name="joint_tool0" type="fixed">
       <origin xyz="0 0 0.015" rpy="0 0 0" />
       <parent link="Link6" />
       <child link="tool0" />
-    </joint>
+    </joint> -->
     <!-- tool_frame -->
     <link name="ee_link"/>
@@ -463,9 +463,9 @@
     </joint>
     <!-- camera -->
-    <!-- <xacro:include filename="$(find rm_description)/urdf/sensors/_d415.urdf.xacro"/>
-    <xacro:sensor_d415  parent="tool0">
-          <origin xyz="-0.05 0 0"
+    <xacro:include filename="$(find rm_description)/urdf/sensors/_d415.urdf.xacro"/>
+    <xacro:sensor_d415  parent="Link6" >
+          <origin xyz="-0.05 0 0.015"
                   rpy="0 -1.57 0" />
-    </xacro:sensor_d415> -->
+    </xacro:sensor_d415>
     <!-- gripper -->
     <link name="gripper_link">
@@ -481,14 +481,14 @@
         </geometry>
       </visual>
-      <collision>
+      <!-- <collision>
         <origin xyz="0 0 0.055" rpy="0 0 0"/>
         <geometry>
             <box size="0.035 0.05 0.11"/>
         </geometry>
-      </collision>
+      </collision> -->
     </link>
     <joint name="joint_gripper" type="fixed">
-      <origin xyz="0 0 0" rpy="0 0 0" />
-      <parent link="tool0" />
+      <origin xyz="0 0 0.015" rpy="0 0 0" />
+      <parent link="Link6" />
       <child link="gripper_link" />
     </joint>

File: src/rm_robot/rm_description/urdf/RM65/rm_65_plus.urdf.xacro (robot description, xacro)
@@ -456,9 +456,9 @@
   </joint>
   <!-- camera -->
-  <!-- <xacro:include filename="$(find rm_description)/urdf/sensors/_d415.urdf.xacro"/>
+  <xacro:include filename="$(find rm_description)/urdf/sensors/_d415.urdf.xacro"/>
     <xacro:sensor_d415  parent="tool0">
         <origin xyz="-0.05 0 0"
                 rpy="0 -1.57 0" />
-  </xacro:sensor_d415> -->
+  </xacro:sensor_d415>
   <!-- gripper -->
   <link name="gripper_link">

File: src/rm_robot/rm_moveit_config/rm_65_moveit_config/config/gazebo_base.urdf (robot description, URDF)
Before this commit: robot base, 17 links, 16 joints
Links:
- added link camera_bottom_screw_frame
- added link camera_link, mass 0.072; collision box size=0.02005 0.099 0.023; visual mesh filename=package://realsense2_description/meshes/d415.stl
- link gripper_link: mass 0.1 -> None; geometry visual box size=0.035 0.05 0.11
Joints:
- added joint camera_joint: type fixed, parent tool0, child camera_bottom_screw_frame, origin xyz=-0.05 0 0 rpy=0 -1.57 0
- added joint camera_link_joint: type fixed, parent camera_bottom_screw_frame, child camera_link, origin xyz=0 0.02 0.0115 rpy=0 0 0
