Commit message: 添加gripper_rviz

File: src/rm_robot/rm_description/urdf/RM65/rm_65_plus.urdf.xacro (robot description, xacro)
@@ -451,7 +451,14 @@
   <link name="tool0"/>
   <joint name="joint_tool0" type="fixed">
-    <origin xyz="0 0 0.01" rpy="0 0 0" />
+    <origin xyz="0 0 0.015" rpy="0 0 0" />
     <parent link="Link6" />
     <child link="tool0" />
+  </joint>
+  <!-- tool_frame -->
+  <link name="ee_link"/>
+  <joint name="joint_ee_link" type="fixed">
+    <origin xyz="0 0 0.14" rpy="0 0 0" />
+    <parent link="Link6" />
+    <child link="ee_link" />
   </joint>
   <!-- camera -->

File: src/rm_robot/rm_moveit_config/rm_65_moveit_config/config/gazebo_rm_65.urdf (robot description, URDF)
Before this commit: robot rm_65, 9 links, 8 joints
Links:
- added link camera_bottom_screw_frame
- added link camera_link, mass 0.072; collision box size=0.02005 0.099 0.023; visual mesh filename=package://realsense2_description/meshes/d415.stl
- added link ee_link
- added link finger1, mass 0.1; collision box size=0.046 0.003 0.065; visual box size=0.046 0.003 0.065
- added link finger2, mass 0.1; collision box size=0.046 0.003 0.065; visual box size=0.046 0.003 0.065
- added link gripper_link, mass 0.1; collision box size=0.035 0.05 0.11; visual box size=0.035 0.05 0.11
- added link tool0
Joints:
- added joint camera_joint: type fixed, parent tool0, child camera_bottom_screw_frame, origin xyz=-0.05 0 0 rpy=0 -1.57 0
- added joint camera_link_joint: type fixed, parent camera_bottom_screw_frame, child camera_link, origin xyz=0 0.02 0.0115 rpy=0 0 0
- added joint joint_ee_link: type fixed, parent Link6, child ee_link, origin xyz=0 0 0.15 rpy=0 0 0
- added joint joint_finger1: type fixed, parent gripper_link, child finger1, origin xyz=0 0.0265 0.11 rpy=0 0 0
- added joint joint_finger2: type fixed, parent gripper_link, child finger2, origin xyz=0 -0.0265 0.11 rpy=0 0 0
- added joint joint_gripper: type fixed, parent tool0, child gripper_link, origin xyz=0 0 0 rpy=0 0 0
- added joint joint_tool0: type fixed, parent Link6, child tool0, origin xyz=0 0 0.01 rpy=0 0 0

Commit message: test1

File: src/rm_robot/rm_description/urdf/RM65/rm_65_plus.urdf.xacro (robot description, xacro)
@@ -18,5 +18,5 @@
     </inertial>
   </xacro:macro>
-  <link name="dummy">
+  <link name="world">
   </link>
   <!-- ///////////////////////////////////////   bottom_joint   ////////////////////////////////////////// -->
@@ -91,5 +91,5 @@
   </gazebo>
   <joint name="dummy_joint" type="fixed">
-    <parent link="dummy" />
+    <parent link="world" />
     <child link="base_link" />
   </joint>
@@ -463,9 +463,9 @@
   </joint>
   <!-- camera -->
-  <xacro:include filename="$(find rm_description)/urdf/sensors/_d415.urdf.xacro"/>
+  <!-- <xacro:include filename="$(find rm_description)/urdf/sensors/_d415.urdf.xacro"/>
     <xacro:sensor_d415  parent="tool0">
         <origin xyz="-0.05 0 0"
                 rpy="0 -1.57 0" />
-  </xacro:sensor_d415>
+  </xacro:sensor_d415> -->
   <!-- gripper -->
   <link name="gripper_link">

File: src/rm_robot/rm_description/urdf/sensors/_d415.urdf.xacro (robot description, xacro)
@@ -8,6 +8,6 @@
 <robot name="sensor_d415" xmlns:xacro="http://ros.org/wiki/xacro">
   <!-- Includes -->
-  <xacro:include filename="$(find rm_description)/urdf/sensors/_materials.urdf.xacro" />
-  <xacro:include filename="$(find rm_description)/urdf/sensors/_usb_plug.urdf.xacro" />
+  <xacro:include filename="$(find realsense2_description)/urdf/_materials.urdf.xacro" />
+  <xacro:include filename="$(find realsense2_description)/urdf/_usb_plug.urdf.xacro" />
   <xacro:macro name="sensor_d415" params="parent *origin  name:=camera  use_nominal_extrinsics:=false add_plug:=false use_mesh:=true">
     <xacro:property name="M_PI" value="3.1415926535897931" />
@@ -36,10 +36,10 @@
     </joint>
     <link name="${name}_bottom_screw_frame"/>
-    <joint name="${name}_link1_joint" type="fixed">
+    <joint name="${name}_link_joint" type="fixed">
       <origin xyz="0 ${d415_cam_depth_py} ${d415_cam_depth_pz}" rpy="0 0 0"/>
       <parent link="${name}_bottom_screw_frame"/>
-      <child link="${name}_link1" />
+      <child link="${name}_link" />
     </joint>
-    <link name="${name}_link1">
+    <link name="${name}_link">
       <visual>
         <xacro:if value="${use_mesh}">
@@ -75,5 +75,5 @@
       <joint name="${name}_depth_joint" type="fixed">
         <origin xyz="0 0 0" rpy="0 0 0"/>
-        <parent link="${name}_link1"/>
+        <parent link="${name}_link"/>
         <child link="${name}_depth_frame" />
       </joint>
@@ -88,5 +88,5 @@
       <joint name="${name}_infra1_joint" type="fixed">
         <origin xyz="0 ${d415_cam_depth_to_infra1_offset} 0" rpy="0 0 0" />
-        <parent link="${name}_link1" />
+        <parent link="${name}_link" />
         <child link="${name}_infra1_frame" />
       </joint>
@@ -101,5 +101,5 @@
       <joint name="${name}_infra2_joint" type="fixed">
         <origin xyz="0 ${d415_cam_depth_to_infra2_offset} 0" rpy="0 0 0" />
-        <parent link="${name}_link1" />
+        <parent link="${name}_link" />
         <child link="${name}_infra2_frame" />
       </joint>
@@ -114,5 +114,5 @@
       <joint name="${name}_color_joint" type="fixed">
         <origin xyz="0 ${d415_cam_depth_to_color_offset} 0" rpy="0 0 0" />
-        <parent link="${name}_link1" />
+        <parent link="${name}_link" />
         <child link="${name}_color_frame" />
       </joint>
@@ -126,5 +126,5 @@
     </xacro:if>
     <xacro:if value="${add_plug}">
-      <xacro:usb_plug parent="${name}_link1" name="${name}_usb_plug">
+      <xacro:usb_plug parent="${name}_link" name="${name}_usb_plug">
         <origin xyz="${d415_cam_mount_from_center_offset - 0.01587} ${-d415_cam_depth_py - 0.0358} 0" rpy="0 0 0"/>
       </xacro:usb_plug>

File: src/rm_robot/rm_moveit_config/rm_65_moveit_config/config/gazebo_rm_65.urdf (robot description, URDF)
Before this commit: robot rm_65, 16 links, 15 joints
Links:
- removed link camera_bottom_screw_frame
- removed link camera_link1
- removed link dummy
- added link world
Joints:
- removed joint camera_joint
- removed joint camera_link1_joint
- joint dummy_joint: parent dummy -> world

Commit message: update

File: src/rm_robot/rm_description/urdf/RM65/rm_65_plus.urdf.xacro (robot description, xacro)
@@ -21,5 +21,5 @@
   </link>
   <!-- ///////////////////////////////////////   bottom_joint   ////////////////////////////////////////// -->
-  <joint name="bottom_joint" type="fixed">
+  <!-- <joint name="bottom_joint" type="fixed">
     <origin xyz="0 0 0" rpy="0 0 0" />
     <parent link="base_link"/>
@@ -43,7 +43,7 @@
     </collision>
     <xacro:Box_inertial_matrix m="500" l="1" w="1" h="0.02"/>
-  </link>
-  <link
-    name="base_link">
+  </link> -->
+  <link
+    name="base_link_rm">
     <inertial>
       <origin
@@ -84,5 +84,5 @@
     </collision>
   </link>
-  <gazebo reference="base_link">
+  <gazebo reference="base_link_rm">
     <mu1 value="200000.0"/>
     <mu2 value="200000.0"/>
@@ -92,5 +92,5 @@
   <joint name="dummy_joint" type="fixed">
     <parent link="world" />
-    <child link="base_link" />
+    <child link="base_link_rm" />
   </joint>
   <link
@@ -141,5 +141,5 @@
       rpy="0 0 0" />
     <parent
-      link="base_link" />
+      link="base_link_rm" />
     <child
       link="Link1" />

File: src/rm_robot/rm_moveit_config/rm_65_moveit_config/config/gazebo_rm_65.urdf (robot description, URDF)
Before this commit: robot rm_65, 14 links, 13 joints
Links:
- removed link base_link
- removed link bottom_link
- added link base_link_rm, mass 0.841070778135659; collision mesh filename=package://rm_description/meshes/RM65/base_link.STL; visual mesh filename=package://rm_description/meshes/RM65/base_link.STL
Joints:
- removed joint bottom_joint
- joint dummy_joint: child base_link -> base_link_rm
- joint joint1: parent base_link -> base_link_rm

Commit message: color_detect&transform

File: src/rm_robot/rm_description/urdf/RM65/rm_65_plus.urdf.xacro (robot description, xacro)
@@ -463,9 +463,9 @@
   </joint>
   <!-- camera -->
-  <!-- <xacro:include filename="$(find rm_description)/urdf/sensors/_d415.urdf.xacro"/>
+  <xacro:include filename="$(find rm_description)/urdf/sensors/_d415.urdf.xacro"/>
     <xacro:sensor_d415  parent="tool0">
         <origin xyz="-0.05 0 0"
                 rpy="0 -1.57 0" />
-  </xacro:sensor_d415> -->
+  </xacro:sensor_d415>
   <!-- gripper -->
   <link name="gripper_link">

File: src/rm_robot/rm_moveit_config/rm_65_moveit_config/config/gazebo_rm_65.urdf (robot description, URDF)
Before this commit: robot rm_65, 13 links, 12 joints
Links:
- added link camera_bottom_screw_frame
- added link camera_link, mass 0.072; collision box size=0.02005 0.099 0.023; visual mesh filename=package://realsense2_description/meshes/d415.stl
Joints:
- added joint camera_joint: type fixed, parent tool0, child camera_bottom_screw_frame, origin xyz=-0.05 0 0 rpy=0 -1.57 0
- added joint camera_link_joint: type fixed, parent camera_bottom_screw_frame, child camera_link, origin xyz=0 0.02 0.0115 rpy=0 0 0

Commit message: 1

File: src/rm_robot/rm_description/urdf/RM65/rm_65_plus.urdf.xacro (robot description, xacro)
@@ -494,5 +494,5 @@
   </joint>
   <!-- finger1 -->
-  <link name="finger1">
+  <!-- <link name="finger1">
     <visual>
       <origin xyz="0 0 0.0325" rpy="0 0 0"/>
@@ -517,7 +517,7 @@
     <parent link="gripper_link" />
     <child link="finger1" />
-  </joint>
+  </joint> -->
   <!-- finger2 -->
-  <link name="finger2">
+  <!-- <link name="finger2">
     <visual>
       <origin xyz="0 0 0.0325" rpy="0 0 0"/>
@@ -542,5 +542,5 @@
     <parent link="gripper_link" />
     <child link="finger2" />
-  </joint>
+  </joint> -->
   <!-- Transmissions for ROS Control -->
   <xacro:macro name="transmission_block" params="joint_name">

Commit message: chessboard_detect

File: src/rm_robot/rm_description/urdf/RM65/rm_65_plus.urdf.xacro (robot description, xacro)
@@ -457,6 +457,6 @@
   <!-- camera -->
   <xacro:include filename="$(find rm_description)/urdf/sensors/_d415.urdf.xacro"/>
-    <xacro:sensor_d415  parent="tool0">
-        <origin xyz="-0.05 0 0"
+    <xacro:sensor_d415  parent="Link6">
+        <origin xyz="-0.05 0 0.015"
                 rpy="0 -1.57 0" />
   </xacro:sensor_d415>
